File: CAD/Eagle/LandCruiser-Controller_1V0.sch (EAGLE design)
At the start: 65 parts, among them K311 V23086C1001A403, K312 V23086C1001A403, K313 V23086C1001A403, K314 V23086C1001A403, K315 V23086C1001A403, U101 MEGA8-P, U221 SN75240, U301 MIC2981/2982SO18W, U501 MAX232_SOIC16, U611 LM7805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

Commit message: HW_V1.0 - fuse drillings added - V1.0 finished and ordered
Parts:
- renumbered U611 to IC611
Changed lines of the file:
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@@
 <part name="P+12V_601" library="df4iah_supply" deviceset="+12V" device=""/>
 <part name="+5V_611" library="df4iah_supply" deviceset="+5V" device=""/>
-<part name="U611" library="df4iah_powersupply" deviceset="78*" device="T" technology="05" value="LM7805"/>
+<part name="IC611" library="df4iah_powersupply" deviceset="78*" device="T" technology="05" value="LM7805"/>
 <part name="GND601" library="df4iah_supply" deviceset="GND" device=""/>
 <part name="C621" library="rcl" deviceset="C-EU" device="C0805" value="22uF"/>
@@
 <instance part="P+12V_601" gate="1" x="203.2" y="106.68" rot="R270"/>
 <instance part="+5V_611" gate="G$1" x="203.2" y="96.52" rot="R270"/>
-<instance part="U611" gate="A1" x="149.86" y="96.52"/>
+<instance part="IC611" gate="A1" x="149.86" y="96.52"/>
 <instance part="GND601" gate="1" x="149.86" y="68.58"/>
 <instance part="C621" gate="G$1" x="177.8" y="86.36"/>
@@
 <wire x1="106.68" y1="73.66" x2="106.68" y2="81.28" width="0.1524" layer="91"/>
 <junction x="119.38" y="73.66"/>
-<pinref part="U611" gate="A1" pin="GND"/>
+<pinref part="IC611" gate="A1" pin="GND"/>
 <pinref part="C602" gate="G$1" pin="2"/>
 <wire x1="132.08" y1="73.66" x2="132.08" y2="81.28" width="0.1524" layer="91"/>
@@
 <segment>
 <pinref part="+5V_611" gate="G$1" pin="+5V"/>
-<pinref part="U611" gate="A1" pin="VO"/>
+<pinref part="IC611" gate="A1" pin="VO"/>
 <wire x1="200.66" y1="96.52" x2="177.8" y2="96.52" width="0.1524" layer="91"/>
 <pinref part="C621" gate="G$1" pin="1"/>
@@
 <pinref part="D601" gate="G$1" pin="C"/>
 <pinref part="C601" gate="G$1" pin="+"/>
-<pinref part="U611" gate="A1" pin="VI"/>
+<pinref part="IC611" gate="A1" pin="VI"/>
 <wire x1="119.38" y1="96.52" x2="132.08" y2="96.52" width="0.1524" layer="91"/>
 <wire x1="132.08" y1="96.52" x2="139.7" y2="96.52" width="0.1524" layer="91"/>
